File: Schematic/mcremote.brd (EAGLE design)
At the start: 60.6 x 25.4 mm, 30 parts, among them IC1 MEGA328P, T1 2N3904

Commit message: Add audio source select button to schematic + PCB
Parts:
- added C8: 100n, rcl:C025-024X044
- added D5: SB120, diode:DO41-7.6
- added X_SW4: 22-23-2021, con-molex:22-23-2021
Connections:
- net N$11 renamed RX
- net N$12 renamed TX
- new net A_SRC: C8.1, D5.C, IC1.23, X_SW4.1
- net GND: now also C8.2, X_SW4.2
- net INT: now also D5.A
Routing:
- net INT: track 12.7 -> 64.4 mm, vias 0 -> 1
- net A_SRC: track 0.00 -> 47.8 mm
- net GND: track 146.2 -> 158.4 mm
Changed lines of the file:
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@@
 <attribute name="VALUE" x="60.071" y="7.62" size="1.27" layer="27" ratio="10" rot="R90"/>
+</element>
+<element name="X_SW4" library="con-molex" library_urn="urn:adsk.eagle:library:165" package="22-23-2021" package3d_urn="urn:adsk.eagle:package:8078633/1" value="22-23-2021" x="57.15" y="22.86" smashed="yes" rot="R270">
+<attribute name="MF" value="MOLEX" x="57.15" y="22.86" size="1.778" layer="27" rot="R270" display="off"/>
+<attribute name="MPN" value="22-23-2021" x="57.15" y="22.86" size="1.778" layer="27" rot="R270" display="off"/>
+<attribute name="NAME" x="60.96" y="25.4" size="1.016" layer="25" ratio="10" rot="R270"/>
+<attribute name="OC_FARNELL" value="1462926" x="57.15" y="22.86" size="1.778" layer="27" rot="R270" display="off"/>
+<attribute name="OC_NEWARK" value="25C3832" x="57.15" y="22.86" size="1.778" layer="27" rot="R270" display="off"/>
+<attribute name="POPULARITY" value="40" x="57.15" y="22.86" size="1.778" layer="27" rot="R270" display="off"/>
+<attribute name="VALUE" x="52.07" y="25.4" size="1.016" layer="27" ratio="10" rot="R270"/>
+</element>
+<element name="D5" library="diode" library_urn="urn:adsk.eagle:library:210" package="DO41-7.6" package3d_urn="urn:adsk.eagle:package:43421/1" value="SB120" x="45.72" y="24.13" smashed="yes" rot="R180">
+<attribute name="NAME" x="47.752" y="22.479" size="1.27" layer="25" ratio="10" rot="R180"/>
+<attribute name="VALUE" x="47.752" y="26.924" size="1.27" layer="27" ratio="10" rot="R180"/>
+</element>
+<element name="C8" library="rcl" library_urn="urn:adsk.eagle:library:334" package="C025-024X044" package3d_urn="urn:adsk.eagle:package:23630/1" value="100n" x="52.07" y="22.86" smashed="yes" rot="R270">
+<attribute name="NAME" x="53.467" y="24.638" size="1.27" layer="25" ratio="10" rot="R270"/>
+<attribute name="SPICEPREFIX" value="C" x="52.07" y="22.86" size="1.778" layer="27" rot="R270" display="off"/>
+<attribute name="VALUE" x="49.403" y="24.638" size="1.27" layer="27" ratio="10" rot="R270"/>
 </element>
 </elements>
@@
 <wire x1="41.91" y1="18.796" x2="42.672" y2="19.558" width="0.6096" layer="16"/>
 <wire x1="41.91" y1="8.89" x2="41.91" y2="18.796" width="0.6096" layer="16"/>
+<contactref element="X_SW4" pad="2"/>
+<contactref element="C8" pad="2"/>
+<wire x1="57.15" y1="21.59" x2="52.07" y2="21.59" width="0.6604" layer="16"/>
+<wire x1="52.07" y1="21.59" x2="49.53" y2="21.59" width="0.6604" layer="16"/>
+<wire x1="49.53" y1="21.59" x2="47.498" y2="19.558" width="0.6604" layer="16"/>
+<wire x1="47.498" y1="19.558" x2="45.72" y2="19.558" width="0.6604" layer="16"/>
 </signal>
 <signal name="+6V">
@@
 <wire x1="49.53" y1="-2.54" x2="52.07" y2="0" width="0.6096" layer="1"/>
 <wire x1="52.07" y1="0" x2="52.07" y2="1.27" width="0.6096" layer="1"/>
-<wire x1="52.07" y1="1.27" x2="52.07" y2="6.35" width="0.6096" layer="1"/>
-<wire x1="45.72" y1="12.7" x2="52.07" y2="6.35" width="0.6096" layer="1"/>
-<wire x1="45.72" y1="16.002" x2="45.72" y2="12.7" width="0.6096" layer="1"/>
+<wire x1="52.07" y1="1.27" x2="52.07" y2="7.62" width="0.6096" layer="1"/>
+<wire x1="45.72" y1="13.97" x2="52.07" y2="7.62" width="0.6096" layer="1"/>
+<wire x1="45.72" y1="16.002" x2="45.72" y2="13.97" width="0.6096" layer="1"/>
 </signal>
 <signal name="+3V3">
@@
 <wire x1="8.89" y1="3.81" x2="8.89" y2="6.35" width="0.6096" layer="16"/>
 <wire x1="8.89" y1="6.35" x2="8.89" y2="8.89" width="0.6096" layer="16"/>
-<wire x1="8.89" y1="8.89" x2="8.89" y2="13.97" width="0.6096" layer="16"/>
+<wire x1="8.89" y1="8.89" x2="8.89" y2="10.16" width="0.6096" layer="16"/>
+<contactref element="D5" pad="A"/>
+<wire x1="45.593" y1="11.90345" x2="44.92345" y2="12.573" width="0.6604" layer="1"/>
+<wire x1="45.593" y1="10.95655" x2="45.593" y2="11.90345" width="0.6604" layer="1"/>
+<wire x1="18.50290625" y1="10.2108" x2="18.45210625" y2="10.16" width="0.6604" layer="1"/>
+<wire x1="18.45210625" y1="10.16" x2="8.89" y2="10.16" width="0.6604" layer="1"/>
+<wire x1="45.593" y1="10.95655" x2="44.84725" y2="10.2108" width="0.6604" layer="1"/>
+<wire x1="44.84725" y1="10.2108" x2="18.50290625" y2="10.2108" width="0.6604" layer="1"/>
+<via x="8.89" y="10.16" extent="1-16" drill="0.35"/>
+<wire x1="8.89" y1="10.16" x2="8.89" y2="13.97" width="0.6604" layer="16"/>
+<wire x1="43.18" y1="14.31645" x2="44.92345" y2="12.573" width="0.6604" layer="1"/>
+<wire x1="41.91" y1="24.13" x2="43.18" y2="22.86" width="0.6604" layer="1"/>
+<wire x1="43.18" y1="22.86" x2="43.18" y2="14.31645" width="0.6604" layer="1"/>
 </signal>
 <signal name="A_PWR">
@@
 <wire x1="1.27" y1="16.51" x2="1.27" y2="13.97" width="0.6096" layer="16"/>
 </signal>
-<signal name="N$11">
+<signal name="RX">
 <contactref element="IC1" pad="2"/>
 <contactref element="TP_RX" pad="TP"/>
 <wire x1="3.81" y1="13.97" x2="3.81" y2="11.43" width="0.6096" layer="16"/>
 </signal>
-<signal name="N$12">
+<signal name="TX">
 <contactref element="IC1" pad="3"/>
 <contactref element="TP_TX" pad="TP"/>
@@
 <wire x1="24.13" y1="24.13" x2="24.13" y2="21.59" width="0.6096" layer="16"/>
 </signal>
+<signal name="A_SRC">
+<contactref element="C8" pad="1"/>
+<contactref element="D5" pad="C"/>
+<contactref element="IC1" pad="23"/>
+<contactref element="X_SW4" pad="1"/>
+<wire x1="57.15" y1="24.13" x2="52.07" y2="24.13" width="0.6604" layer="16"/>
+<wire x1="52.07" y1="24.13" x2="49.53" y2="24.13" width="0.6604" layer="16"/>
+<wire x1="49.53" y1="24.13" x2="46.99" y2="26.67" width="0.6604" layer="1"/>
+<wire x1="46.99" y1="26.67" x2="16.51" y2="26.67" width="0.6604" layer="1"/>
+<wire x1="16.51" y1="26.67" x2="13.97" y2="24.13" width="0.6604" layer="1"/>
+<wire x1="13.97" y1="24.13" x2="13.97" y2="21.59" width="0.6604" layer="1"/>
+</signal>
 </signals>
