File: Schematic/mcremote.sch (EAGLE design)
At the start: 30 parts, among them IC1 MEGA328P, T1 2N3904

Commit message: Add audio source select button to schematic + PCB
Parts:
- added C8: 100n, rcl:C-EU025-024X044
- added D5: SB120, diode:DIODE-DO41-7.6
- added X_SW4: 22-23-2021, con-molex:22-23-2021
Connections:
- net N$11 renamed RX
- net N$12 renamed TX
- new net A_SRC: C8.1, D5.C, IC1.PC0(ADC0), X_SW4-1.S
- net GND: now also C8.2, X_SW4-2.S
- net INT: now also D5.A
Changed lines of the file:
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@@
 <part name="FRAME1" library="frames" library_urn="urn:adsk.eagle:library:229" deviceset="A4L-LOC" device=""/>
 <part name="JP1" library="jumper" library_urn="urn:adsk.eagle:library:252" deviceset="JP1E" device="" package3d_urn="urn:adsk.eagle:package:15455/1"/>
+<part name="X_SW4" library="con-molex" library_urn="urn:adsk.eagle:library:165" deviceset="22-23-2021" device="" package3d_urn="urn:adsk.eagle:package:8078633/1"/>
+<part name="D5" library="diode" library_urn="urn:adsk.eagle:library:210" deviceset="DIODE-" device="DO41-7.6" package3d_urn="urn:adsk.eagle:package:43421/1" value="SB120"/>
+<part name="C8" library="rcl" library_urn="urn:adsk.eagle:library:334" deviceset="C-EU" device="025-024X044" package3d_urn="urn:adsk.eagle:package:23630/1" value="100n"/>
+<part name="GND15" library="supply1" library_urn="urn:adsk.eagle:library:371" deviceset="GND" device=""/>
+<part name="GND16" library="supply1" library_urn="urn:adsk.eagle:library:371" deviceset="GND" device=""/>
 </parts>
 <sheets>
@@
 <attribute name="VALUE" x="154.94" y="42.545" size="1.778" layer="96"/>
 </instance>
+<instance part="X_SW4" gate="-1" x="17.78" y="-7.62" smashed="yes" rot="R180">
+<attribute name="NAME" x="15.24" y="-6.858" size="1.524" layer="95" rot="R180"/>
+<attribute name="VALUE" x="18.542" y="-9.017" size="1.778" layer="96" rot="R180"/>
+</instance>
+<instance part="X_SW4" gate="-2" x="17.78" y="-10.16" smashed="yes" rot="R180">
+<attribute name="NAME" x="15.24" y="-9.398" size="1.524" layer="95" rot="R180"/>
+</instance>
+<instance part="D5" gate="G$1" x="33.02" y="-5.08" smashed="yes" rot="R180">
+<attribute name="NAME" x="30.48" y="-5.5626" size="1.778" layer="95" rot="R180"/>
+<attribute name="VALUE" x="30.48" y="-2.7686" size="1.778" layer="96" rot="R180"/>
+</instance>
+<instance part="C8" gate="G$1" x="33.02" y="-15.24" smashed="yes">
+<attribute name="NAME" x="34.544" y="-14.859" size="1.778" layer="95"/>
+<attribute name="VALUE" x="34.544" y="-19.939" size="1.778" layer="96"/>
+</instance>
+<instance part="GND15" gate="1" x="22.86" y="-20.32" smashed="yes">
+<attribute name="VALUE" x="20.32" y="-22.86" size="1.778" layer="96"/>
+</instance>
+<instance part="GND16" gate="1" x="33.02" y="-25.4" smashed="yes">
+<attribute name="VALUE" x="30.48" y="-27.94" size="1.778" layer="96"/>
+</instance>
 </instances>
 <busses>
@@
 <pinref part="GND14" gate="1" pin="GND"/>
 <wire x1="190.5" y1="50.8" x2="190.5" y2="45.72" width="0.1524" layer="91"/>
+</segment>
+<segment>
+<pinref part="GND15" gate="1" pin="GND"/>
+<wire x1="22.86" y1="-10.16" x2="22.86" y2="-17.78" width="0.1524" layer="91"/>
+<pinref part="X_SW4" gate="-2" pin="S"/>
+<wire x1="22.86" y1="-10.16" x2="20.32" y2="-10.16" width="0.1524" layer="91"/>
+</segment>
+<segment>
+<pinref part="C8" gate="G$1" pin="2"/>
+<pinref part="GND16" gate="1" pin="GND"/>
+<wire x1="33.02" y1="-20.32" x2="33.02" y2="-22.86" width="0.1524" layer="91"/>
 </segment>
 </net>
@@
 <label x="215.9" y="127" size="1.27" layer="95" xref="yes"/>
 </segment>
+<segment>
+<pinref part="D5" gate="G$1" pin="A"/>
+<wire x1="35.56" y1="-5.08" x2="50.8" y2="-5.08" width="0.1524" layer="91"/>
+<label x="50.8" y="-5.08" size="1.27" layer="95" xref="yes"/>
+</segment>
 </net>
 <net name="A_PWR" class="0">
@@
 </segment>
 </net>
-<net name="N$11" class="0">
+<net name="RX" class="0">
 <segment>
 <pinref part="IC1" gate="G$1" pin="PD0(RXD)"/>
@@
 </segment>
 </net>
-<net name="N$12" class="0">
+<net name="TX" class="0">
 <segment>
 <pinref part="IC1" gate="G$1" pin="PD1(TXD)"/>
@@
 </segment>
 </net>
+<net name="A_SRC" class="0">
+<segment>
+<wire x1="25.4" y1="-7.62" x2="33.02" y2="-7.62" width="0.1524" layer="91"/>
+<wire x1="50.8" y1="-7.62" x2="33.02" y2="-7.62" width="0.1524" layer="91"/>
+<pinref part="C8" gate="G$1" pin="1"/>
+<wire x1="33.02" y1="-12.7" x2="33.02" y2="-7.62" width="0.1524" layer="91"/>
+<junction x="33.02" y="-7.62"/>
+<pinref part="D5" gate="G$1" pin="C"/>
+<wire x1="30.48" y1="-5.08" x2="25.4" y2="-5.08" width="0.1524" layer="91"/>
+<wire x1="25.4" y1="-5.08" x2="25.4" y2="-7.62" width="0.1524" layer="91"/>
+<label x="50.8" y="-7.62" size="1.27" layer="95" xref="yes"/>
+<pinref part="X_SW4" gate="-1" pin="S"/>
+<wire x1="20.32" y1="-7.62" x2="25.4" y2="-7.62" width="0.1524" layer="91"/>
+<junction x="25.4" y="-7.62"/>
+</segment>
+<segment>
+<pinref part="IC1" gate="G$1" pin="PC0(ADC0)"/>
+<wire x1="198.12" y1="154.94" x2="215.9" y2="154.94" width="0.1524" layer="91"/>
+<label x="215.9" y="154.94" size="1.27" layer="95" xref="yes"/>
+</segment>
+</net>
 </nets>
 </sheet>
 </sheets>
-<errors>
-</errors>
 </schematic>
 </drawing>
